File: haven-c-badges.kicad_pcb (KiCad board)
At the start: 2 copper layers, 241.3 x 99.2 mm, 15 parts, among them U1 NT3H2111W0FHKH

Commit message: FIxed the daven issues + deprecated components
- Fixed daven potential mishap
- Moved the components to the right places
- Set the other versions aside
Parts:
- added F.Cu, F.mask: LOGO, LOGO, F.Cu at (177.6, 95.5)
- added Logo Copper: LOGO, LOGO, B.Cu at (194.6, 70.3)
- added Logo Mask: LOGO, LOGO, B.Cu at (194.6, 70.2)
- added Logo Shadow Copper: LOGO, LOGO, F.Cu at (177.5, 76.5)
- added LogoShadowMask: LOGO, LOGO, F.Cu at (177.5, 76.5)
- added UV Print Silkscreen Guide: LOGO, LOGO, F.Cu at (177.6, 95.5)
- moved BottomSilkscreen 95.7 mm to (85.7, 97.2)
- moved REF** 95.7 mm to (85.5, 54.1)
- moved UV Print Guide 95.6 mm to (85.9, 96.9)
- moved F.Soldermask 72.5 mm to (247.1, 95.5)
- moved B.Silkscreen 72.5 mm to (177.6, 95.3)
- moved C1 72.5 mm to (177.6, 133.9)
- moved D1 72.5 mm to (177.6, 137.6)
- moved L1 72.5 mm to (177.6, 116.2)
- moved R1 72.5 mm to (179.6, 133.1)
- moved REF** 72.5 mm to (177.5, 54.1)
- moved U1 72.5 mm to (177.7, 132.3)
- moved REF** 39.3 mm to (26.5, 73.0)
- moved F.Gold 3.67 mm to (246.5, 95.1)
- moved F.Mask 3.67 mm to (246.5, 95.1)
- moved 98.5 Import F.Silkscreen 3.01 mm to (247.1, 95.5)
Other:
- board size 241.3 x 99.2 mm -> 153.8 x 99.2 mm

Commit message: Removed the older versions & gerbers
- only 1 board is left now
- Removed the older failed versions in the side
- deleted the gerbers for a refresh
Parts:
- removed 98.5 Import F.Silkscreen: LOGO, LOGO
- removed BottomSilkscreen, F.Gold, F.Mask, F.Soldermask: LOGO, LOGO
- removed REF** (x2): Lanyard_hole2, Lanyard_hole2
- removed UV Print Guide: LOGO, LOGO
- 4mm Lanyard Hole: renamed from REF**
- moved D1 1.70 mm to (177.6, 139.3)
Routing:
- net Net-(D1-K): track 6.00 -> 7.70 mm
- net Net-(D1-A): track 4.11 -> 5.81 mm
Other:
- board size 153.8 x 99.2 mm -> 61.3 x 97 mm
- board text removed: "0.125"
